Commit message: 更新pick and place的默认输入，以及对应的判断条件

File: unilabos/device_mesh/devices/agilent_biotek_406_fx/macro_device.xacro (robot description, xacro)
@@ -73,10 +73,10 @@
         </material>
       </visual>
-      <collision>
+      <!-- <collision>
         <origin xyz="0 0 ${height / 2.0}" rpy="0 0 0"/>
         <geometry>
           <box size="${width} ${depth} ${height}"/>
         </geometry>
-      </collision>
+      </collision> -->
     </link>
     <link name="${station_name}${device_name}plate_carrier_link">

File: unilabos/device_mesh/devices/applied_biosystems_seqstudio_genetic_analyzer/macro_device.xacro (robot description, xacro)
@@ -42,5 +42,5 @@
       </visual>
       <!-- 将机身碰撞拆分为后壳、前侧壁和前上罩，保持前向 sample/cartridge 装载走廊敞开。 -->
-      <collision>
+      <!-- <collision>
         <origin xyz="0 ${rear_body_center_y} ${height / 2.0}" rpy="0 0 0"/>
         <geometry>
@@ -65,5 +65,5 @@
           <box size="${width} ${front_corridor_depth} ${height - front_corridor_height}"/>
         </geometry>
-      </collision>
+      </collision> -->
     </link>
     <!-- 内部样本板中心位；SeqStudio 支持 96 孔板和 8 联管。 -->

File: unilabos/device_mesh/devices/bd_facsmelody/macro_device.xacro (robot description, xacro)
@@ -85,5 +85,5 @@
       </visual>
       <!-- Keep the sorter shell conservative while leaving the front chamber and rear service hatch open. -->
-      <collision>
+      <!-- <collision>
         <origin xyz="0 ${middle_body_center_y} ${height / 2.0}" rpy="0 0 0"/>
         <geometry>
@@ -132,5 +132,5 @@
           <box size="${rear_corridor_width} ${rear_corridor_depth} ${height - rear_corridor_bottom_z - rear_corridor_height}"/>
         </geometry>
-      </collision>
+      </collision> -->
     </link>
     <!-- Estimated front-left sample loading region for 5 mL tubes. -->

File: unilabos/device_mesh/devices/bio_shake/macro_device.xacro (robot description, xacro)
@@ -38,5 +38,5 @@
       </visual>
       <!-- Split the simplified collision so the top-contact plate zone is a genuine open recess. -->
-      <collision>
+      <!-- <collision>
         <origin xyz="0 0 ${plate_recess_floor_height / 2.0}" rpy="0 0 0"/>
         <geometry>
@@ -75,5 +75,5 @@
           <box size="${plate_opening_width} ${plate_front_back_wall_depth} ${plate_top_edge_height}"/>
         </geometry>
-      </collision>
+      </collision> -->
     </link>
     <!-- Primary robotic access frame for an ANSI/SLAS microplate on the shaker table. -->

File: unilabos/device_mesh/devices/bio_tek_plate_reader_backend/macro_device.xacro (robot description, xacro)
@@ -42,5 +42,5 @@
       </visual>
       <!-- 主体碰撞拆成后壳、前上壳和左右前侧立柱，避免前部抽屉通道被整块实体封死。 -->
-      <collision>
+      <!-- <collision>
         <origin xyz="0 ${rear_shell_center_y} ${height / 2.0}" rpy="0 0 0"/>
         <geometry>
@@ -65,5 +65,5 @@
           <box size="${front_side_shell_width} ${front_shell_depth} ${front_opening_height}"/>
         </geometry>
-      </collision>
+      </collision> -->
     </link>
     <link name="${station_name}${device_name}service_door_link">
@@ -115,10 +115,10 @@
         </material>
       </visual>
-      <collision>
+      <!-- <collision>
         <origin xyz="0 0 0.005" rpy="0 0 0"/>
         <geometry>
           <box size="0.136 0.093 0.01"/>
         </geometry>
-      </collision>
+      </collision> -->
     </link>
     <joint name="${station_name}${device_name}tray_joint" type="fixed">

File: unilabos/device_mesh/devices/centrifuge/macro_device.xacro (robot description, xacro)
@@ -64,10 +64,10 @@
         </material>
       </visual>
-      <collision>
+      <!-- <collision>
         <origin xyz="0 0 ${height / 2.0}" rpy="0 0 0"/>
         <geometry>
           <box size="${width} ${depth} ${height}"/>
         </geometry>
-      </collision>
+      </collision> -->
     </link>
     <link name="${station_name}${device_name}loading_access_link"/>

File: unilabos/device_mesh/devices/clari_ostar_backend/macro_device.xacro (robot description, xacro)
@@ -45,10 +45,10 @@
         </material>
       </visual>
-      <collision>
+      <!-- <collision>
         <origin xyz="0 0 ${height / 2.0}" rpy="0 0 0"/>
         <geometry>
           <box size="${width} ${depth} ${height}"/>
         </geometry>
-      </collision>
+      </collision> -->
     </link>
     <link name="${station_name}${device_name}socketTypeGenericSbsFootprint"/>

File: unilabos/device_mesh/devices/cytiva_akta_pure/macro_device.xacro (robot description, xacro)
@@ -58,10 +58,10 @@
         </material>
       </visual>
-      <collision>
+      <!-- <collision>
         <origin xyz="0 0 ${height / 2.0}" rpy="0 0 0"/>
         <geometry>
           <box size="${width} ${depth} ${height}"/>
         </geometry>
-      </collision>
+      </collision> -->
     </link>
     <!-- 前侧为主要人工/机械操作面：柱位、阀组件、样品泵、触控面板均位于此侧。 -->

File: unilabos/device_mesh/devices/cytiva_biacore_8k_plus/macro_device.xacro (robot description, xacro)
@@ -95,10 +95,10 @@
         </material>
       </visual>
-      <collision>
+      <!-- <collision>
         <origin xyz="0 0 ${height / 2.0}" rpy="0 0 0"/>
         <geometry>
           <box size="${width} ${depth} ${height}"/>
         </geometry>
-      </collision>
+      </collision> -->
     </link>
     <link name="${station_name}${device_name}sample_hotel_access_link"/>

File: unilabos/device_mesh/devices/cytomat_backend/macro_device.xacro (robot description, xacro)
@@ -66,5 +66,5 @@
         </material>
       </visual>
-      <collision>
+      <!-- <collision>
         <origin xyz="0 ${rear_collision_y} ${height / 2.0}" rpy="0 0 0"/>
         <geometry>
@@ -95,5 +95,5 @@
           <box size="${transfer_opening_side_width} ${front_collision_depth} ${transfer_opening_height}"/>
         </geometry>
-      </collision>
+      </collision> -->
     </link>
     <link name="${station_name}${device_name}loading_tray_link">
@@ -107,10 +107,10 @@
         </material>
       </visual>
-      <collision>
+      <!-- <collision>
         <origin xyz="0 ${loading_tray_collision_y} ${loading_tray_collision_z}" rpy="0 0 0"/>
         <geometry>
           <box size="${loading_tray_collision_width} ${loading_tray_collision_depth} ${loading_tray_collision_height}"/>
         </geometry>
-      </collision>
+      </collision> -->
     </link>
     <joint name="${station_name}${device_name}loading_tray_link_joint" type="fixed">

File: unilabos/device_mesh/devices/hamilton_vantage/macro_device.xacro (robot description, xacro)
@@ -137,5 +137,5 @@
         <material name="hamilton_vantage_internal_dark"/>
       </visual>
-      <collision>
+      <!-- <collision>
         <origin xyz="0 0.080 ${lower_body_height / 2.0}" rpy="0 0 0"/>
         <geometry>
@@ -160,5 +160,5 @@
           <box size="${width * 0.72} 0.120 ${upper_body_height}"/>
         </geometry>
-      </collision>
+      </collision> -->
     </link>
     <link name="${station_name}${device_name}loading_tray_link">
@@ -173,10 +173,10 @@
         </material>
       </visual>
-      <collision>
+      <!-- <collision>
         <origin xyz="0 0 0.015" rpy="0 0 0"/>
         <geometry>
           <box size="0.18 0.14 0.030"/>
         </geometry>
-      </collision>
+      </collision> -->
     </link>
     <joint name="${station_name}${device_name}loading_tray_joint" type="fixed">

File: unilabos/device_mesh/devices/hettich_rotanta_460_robotic/macro_device.xacro (robot description, xacro)
@@ -94,5 +94,5 @@
         </material>
       </visual>
-      <collision>
+      <!-- <collision>
         <origin xyz="0 0 ${top_opening_floor_z / 2.0}" rpy="0 0 0"/>
         <geometry>
@@ -123,5 +123,5 @@
           <box size="${top_side_rim_width} ${top_opening_depth} ${top_opening_height}"/>
         </geometry>
-      </collision>
+      </collision> -->
     </link>
     <!-- Access frames are estimated from official datasheet wording and product imagery:

File: unilabos/device_mesh/devices/molecular_devices_qpix_420/macro_device.xacro (robot description, xacro)
@@ -172,5 +172,5 @@
       </visual>
       <!-- 碰撞几何只保留真实阻挡外壳：开放前工位、deck/worktable 与 SBS 取放区域不再被整机包络盒吞没。 -->
-      <collision>
+      <!-- <collision>
         <origin xyz="0 0 ${plinth_height / 2.0}" rpy="0 0 0"/>
         <geometry>
@@ -213,5 +213,5 @@
           <box size="${control_console_width} ${control_console_depth} ${control_console_height}"/>
         </geometry>
-      </collision>
+      </collision> -->
     </link>
     <!-- 前门对应主要人工开盖访问区域。 -->

File: unilabos/device_mesh/devices/qiagen_qiacube_connect/macro_device.xacro (robot description, xacro)
@@ -81,5 +81,5 @@
         </material>
       </visual>
-      <collision>
+      <!-- <collision>
         <origin xyz="0 0 0.145" rpy="0 0 0"/>
         <geometry>
@@ -104,5 +104,5 @@
           <box size="0.180 0.240 0.230"/>
         </geometry>
-      </collision>
+      </collision> -->
     </link>
     <joint name="${station_name}${device_name}body_link_joint" type="fixed">
@@ -122,10 +122,10 @@
         </material>
       </visual>
-      <collision>
+      <!-- <collision>
         <origin xyz="0 0 0.040" rpy="0 0 0"/>
         <geometry>
           <box size="0.420 0.180 0.080"/>
         </geometry>
-      </collision>
+      </collision> -->
     </link>
     <joint name="${station_name}${device_name}waste_drawer_link_joint" type="fixed">

File: unilabos/device_mesh/devices/tecan_resolvex_a200/macro_device.xacro (robot description, xacro)
@@ -173,5 +173,5 @@
       </visual>
       <!-- 将碰撞拆为下部柜体、上部侧框、后上壳体和前上横梁，保留前部开口与工作平面。 -->
-      <collision>
+      <!-- <collision>
         <origin xyz="0 0 ${lower_body_height / 2.0}" rpy="0 0 0"/>
         <geometry>
@@ -202,5 +202,5 @@
           <box size="${front_lintel_width} ${front_lintel_depth} ${front_lintel_height}"/>
         </geometry>
-      </collision>
+      </collision> -->
     </link>
     <!-- 前部主开口，用于装卸 SPE 板 / 柱架。 -->

File: unilabos/device_mesh/devices/telesis_bio_bioxp_3250/macro_device.xacro (robot description, xacro)
@@ -68,10 +68,10 @@
         </material>
       </visual>
-      <collision>
+      <!-- <collision>
         <origin xyz="0 0 ${height / 2.0}" rpy="0 0 0"/>
         <geometry>
           <box size="${width} ${depth} ${height}"/>
         </geometry>
-      </collision>
+      </collision> -->
     </link>
     <!-- 前门中央附近的主要装载开口参考点。 -->
