Commit message: 修改模型到test环境

File: unilabos/device_mesh/devices/slide_w140/macro_device.xacro (robot description, xacro)
@@ -127,4 +127,11 @@
       <child link="${station_name}${device_name}slide_end"/>
     </joint>
+    <link name="${station_name}${device_name}attach_link"/>
+    <joint name="${station_name}${device_name}attach_joint" type="fixed">
+      <origin rpy="0 0 0" xyz="0 0 0.015"/>
+      <parent link="${station_name}${device_name}slider"/>
+      <child link="${station_name}${device_name}attach_link"/>
+      <axis xyz="0 0 0"/>
+    </joint>
   </xacro:macro>
 </robot>
